File: loadcell/loadcell/loadcell.sch (KiCad schematic (older format))
At the start: 3 parts

Commit message: new files
Parts:
- U?: symbol MCU_Microchip_ATtiny:ATtiny85-20PU -> loadcell-rescue:ATtiny85-20PU-MCU_Microchip_ATtiny
Changed lines of the file:
@@
 EESchema Schematic File Version 4
-LIBS:loadcell-cache
 EELAYER 30 0
 EELAYER END
@@
 $EndDescr
 $Comp
-L MCU_Microchip_ATtiny:ATtiny85-20PU U?
+L loadcell-rescue:ATtiny85-20PU-MCU_Microchip_ATtiny U?
 U 1 1 5D673927
 P 2500 2250
