File: razpi-hat/razpi-hat.sch (KiCad schematic (older format))
At the start: 11 parts, among them J1 Sensor, P1 Conn_02x20_Odd_Even, U1 ATtiny85-20PU, U2 SN75176AP, U3 MPM82

Commit message: new files
Parts:
- added J?: USB_A, symbol Connector:USB_A
- U3: symbol SankenElectric:MPM82 -> razpi-hat-rescue:MPM82-SankenElectric
Connections:
- net +3V3: now also U1.8 (VCC)
- net +5V: now also J?.1 (VBUS); no longer U1.8 (VCC)
- net GND: now also J?.4 (GND), J?.5 (Shield)
- no-connect marks 1 -> 3
Changed lines of the file:
@@
 	5800 4300 5800 4050
-Wire Wire Line
-	5800 4050 4650 4050
 Wire Wire Line
 	3250 4050 3250 4200
@@
 L power:+5V #PWR0101
 U 1 1 5E79E40A
-P 4650 4050
-F 0 "#PWR0101" H 4650 3900 50  0001 C CNN
-F 1 "+5V" H 4665 4223 50  0000 C CNN
-F 2 "" H 4650 4050 50  0001 C CNN
-F 3 "" H 4650 4050 50  0001 C CNN
-	1    4650 4050
-	1    0    0    -1
-$EndComp
-Connection ~ 4650 4050
-Wire Wire Line
-	4650 4050 3250 4050
+P 5800 4050
+F 0 "#PWR0101" H 5800 3900 50  0001 C CNN
+F 1 "+5V" H 5815 4223 50  0000 C CNN
+F 2 "" H 5800 4050 50  0001 C CNN
+F 3 "" H 5800 4050 50  0001 C CNN
+	1    5800 4050
+	1    0    0    -1
+$EndComp
 $Comp
 L power:GND #PWR0102
@@
 $EndComp
 $Comp
-L SankenElectric:MPM82 U3
+L razpi-hat-rescue:MPM82-SankenElectric U3
 U 1 1 5E7D4852
 P 7900 4850
@@
 	8450 4850 8450 4750
 Connection ~ 8450 4750
+$Comp
+L power:+3.3V #PWR?
+U 1 1 5E8FD765
+P 3250 4050
+F 0 "#PWR?" H 3250 3900 50  0001 C CNN
+F 1 "+3.3V" H 3265 4223 50  0000 C CNN
+F 2 "" H 3250 4050 50  0001 C CNN
+F 3 "" H 3250 4050 50  0001 C CNN
+	1    3250 4050
+	1    0    0    -1
+$EndComp
+$Comp
+L Connector:USB_A J?
+U 1 1 5E900888
+P 2550 2450
+F 0 "J?" H 2607 2917 50  0000 C CNN
+F 1 "USB_A" H 2607 2826 50  0000 C CNN
+F 2 "" H 2700 2400 50  0001 C CNN
+F 3 " ~" H 2700 2400 50  0001 C CNN
+	1    2550 2450
+	1    0    0    -1
+$EndComp
+NoConn ~ 2850 2550
+NoConn ~ 2850 2450
+$Comp
+L power:+5V #PWR?
+U 1 1 5E9069A3
+P 3100 2250
+F 0 "#PWR?" H 3100 2100 50  0001 C CNN
+F 1 "+5V" H 3115 2423 50  0000 C CNN
+F 2 "" H 3100 2250 50  0001 C CNN
+F 3 "" H 3100 2250 50  0001 C CNN
+	1    3100 2250
+	1    0    0    -1
+$EndComp
+$Comp
+L power:GND #PWR?
+U 1 1 5E906DAB
+P 2550 3000
+F 0 "#PWR?" H 2550 2750 50  0001 C CNN
+F 1 "GND" H 2555 2827 50  0000 C CNN
+F 2 "" H 2550 3000 50  0001 C CNN
+F 3 "" H 2550 3000 50  0001 C CNN
+	1    2550 3000
+	1    0    0    -1
+$EndComp
+Wire Wire Line
+	2850 2250 3100 2250
+Wire Wire Line
+	2450 2850 2550 2850
+Wire Wire Line
+	2550 3000 2550 2850
+Connection ~ 2550 2850
 $EndSCHEMATC
